File: driver/driver_seperate/driver_seperate.kicad_sch (KiCad schematic)
At the start: 20 parts, among them IC1 MCT8316Z0TQRGFRQ1, J1 Conn_01x08_Pin, J2 Conn_01x05_Pin

Commit message: Add finished pcb
Parts:
- C4: footprint SamacSys_Parts:CAPC6050X350N -> SamacSys_Parts:CAPC6153X500N
- C6: footprint SamacSys_Parts:CAPC6050X350N -> Capacitor_SMD:C_1206_3216Metric
Changed lines of the file:
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@@
       (effects (font (size 1.27 1.27)) (justify left))
     )
-    (property "Footprint" "SamacSys_Parts:CAPC6050X350N" (at 151.638 35.56 0)
+    (property "Footprint" "SamacSys_Parts:CAPC6153X500N" (at 151.638 35.56 0)
       (effects (font (size 1.27 1.27)) hide)
     )
@@
       (effects (font (size 1.27 1.27)) (justify left))
     )
-    (property "Footprint" "SamacSys_Parts:CAPC6050X350N" (at 151.638 64.77 0)
+    (property "Footprint" "Capacitor_SMD:C_1206_3216Metric" (at 151.638 64.77 0)
       (effects (font (size 1.27 1.27)) hide)
     )

Commit message: Add newest version, revision started
Parts:
- removed C1: 47nF, SamacSys_Parts:CAPC3216X180N, symbol Device:C_Small
- removed C2, C5: 1uF, SamacSys_Parts:CAPC3216X178N, symbol Device:C_Small
- removed C3, C7: 0u1F, SamacSys_Parts:CAPC1608X95N, symbol Device:C_Small
- removed C4: >=10uF, SamacSys_Parts:CAPC6153X500N, symbol Device:C_Polarized_Small
- removed C6: 22uF, Capacitor_SMD:C_1206_3216Metric, symbol Device:C_Small
- removed IC1: MCT8316Z0TQRGFRQ1, SamacSys_Parts:QFN50P500X700X100-41N-D, symbol MCT8316Z0TQRGFRQ1:MCT8316Z0TQRGFRQ1
- removed IN+1, IN-1: MountingHole_Pad, MountingHole:MountingHole_2.5mm_Pad, symbol Mechanical:MountingHole_Pad
- removed J1: Conn_01x08_Pin, Connector_PinHeader_1.27mm:PinHeader_1x08_P1.27mm_Vertical, symbol Connector:Conn_01x08_Pin
- removed J2: Conn_01x05_Pin, Connector_PinHeader_1.27mm:PinHeader_1x05_P1.27mm_Vertical, symbol Connector:Conn_01x05_Pin
- removed L1: 47uH, SamacSys_Parts:INDPM7973X540N, symbol Device:L_Small
- removed R1, R2: 1k, Resistor_SMD:R_0603_1608Metric_Pad0.98x0.95mm_HandSolder, symbol Device:R_Small
- removed R3, R4: 5k1, Resistor_SMD:R_0603_1608Metric_Pad0.98x0.95mm_HandSolder, symbol Device:R_Small
- removed R5: 1M, Resistor_SMD:R_0805_2012Metric_Pad1.20x1.40mm_HandSolder, symbol Device:R_Small
- removed R6: 47k, Resistor_SMD:R_0402_1005Metric_Pad0.72x0.64mm_HandSolder, symbol Device:R_Small
- removed R7: 22k, Resistor_SMD:R_0402_1005Metric_Pad0.72x0.64mm_HandSolder, symbol Device:R_Small
- added J1: Conn_01x03, Connector_Molex:Molex_CLIK-Mate_502443-0370_1x03-1MP_P2.00mm_Vertical, symbol Connector_Generic:Conn_01x03
- added J3: Conn_01x07, Connector_Molex:Molex_CLIK-Mate_502382-0770_1x07-1MP_P1.25mm_Vertical, symbol Connector_Generic:Conn_01x07
Connections:
- new net controller/+3V3: J1.2 (Pin_2)
- new net controller/CS: J3.4 (Pin_4)
- new net controller/FGOUT: J3.6 (Pin_6)
- new net controller/GND: J1.3 (Pin_3)
- new net controller/MISO: J3.3 (Pin_3)
- new net controller/MOSI: J3.2 (Pin_2)
- new net controller/NRST: J3.7 (Pin_7)
- new net controller/PWM: J3.5 (Pin_5)
- new net controller/SCK: J3.1 (Pin_1)
- new net controller/VCC: J1.1 (Pin_1)
Other:
- added sheet controller (controller.kicad_sch)
- note added: "2"
- note removed: "5.0V/200mA"
- note removed: "ADVANCE is tied to 22k Ohms to AVDD which gives 4 degree setting. MODE is tied to AVDD which gives PWM Mode; synchronous digital hall input. SLEW is tied ti 47k Ohms resistor to AVDD which gives SLEW=10b. VSEL_BK is set to HI-z wich gives SW_BK 5.0V."
- note removed: "AVDD 3.3V/30mA"
- note removed: "AVDD/2V ILIM disables current limit."
- note removed: "IN+"
- note removed: "IN-"
- note removed: "Motor Driver and Connectors"
- note removed: "Motor hall sensor takes 3.3.. 18V input. Therefore SW_BK is set to 5.0V/200mA."
- note removed: "fgout pwm brake dir nfault"
- note removed: "~3.3/2V"

Commit message: Add start of new design
Parts:
- removed J1: Conn_01x03, Connector_Molex:Molex_CLIK-Mate_502443-0370_1x03-1MP_P2.00mm_Vertical, symbol Connector_Generic:Conn_01x03
- removed J3: Conn_01x07, Connector_Molex:Molex_CLIK-Mate_502382-0770_1x07-1MP_P1.25mm_Vertical, symbol Connector_Generic:Conn_01x07
- added J1: Conn_01x07, Connector_Molex:Molex_KK-254_AE-6410-07A_1x07_P2.54mm_Vertical, symbol Connector_Generic:Conn_01x07
- added J4: Conn_01x02, Connector_Molex:Molex_KK-254_AE-6410-02A_1x02_P2.54mm_Vertical, symbol Connector_Generic:Conn_01x02
Connections:
- net Motor Driver/FGOUT: now also J1.2 (Pin_2)
- net Motor Driver/GND: now also J4.2 (Pin_2)
- net Motor Driver/PWM: now also J1.1 (Pin_1)
- net Motor Driver/VCC: now also J4.1 (Pin_1)
- new net Motor Driver/BRAKE: J1.4 (Pin_4)
- new net Motor Driver/DIR: J1.3 (Pin_3)
- new net Motor Driver/DRVOFF: J1.6 (Pin_6)
- new net Motor Driver/nFault: J1.5 (Pin_5)
- new net Motor Driver/nSleep: J1.7 (Pin_7)
Other:
- sheet controller renamed Motor Driver
- sheet Motor Driver ports: added BRAKE, DIR, DRVOFF, nFault, nSleep; removed +3V3, CS, MISO, MOSI, NRST, SCK
- note added: "DRVOFF turns off motors when HIGH"
- note added: "nfault needs pull up >2.2v at start"
- note added: "nsleep makes device enter sleepmode when LOW"
Changed lines of the file:
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@@
 (kicad_sch (version 20230121) (generator eeschema)
   (paper "A4")
-  (wire (pts (xy 48.641 50.8) (xy 48.641 50.546))
+  (wire (pts (xy 60.96 24.13) (xy 60.96 30.48))
     (stroke (width 0) (type default))
   )
-  (wire (pts (xy 68.961 28.956) (xy 68.961 32.766))
+  (wire (pts (xy 34.29 36.83) (xy 44.45 36.83))
     (stroke (width 0) (type default))
   )
-  (wire (pts (xy 39.37 45.72) (xy 48.641 45.72))
+  (wire (pts (xy 34.29 34.29) (xy 44.45 34.29))
     (stroke (width 0) (type default))
   )
-  (wire (pts (xy 66.421 32.766) (xy 66.421 28.956))
+  (wire (pts (xy 34.29 49.53) (xy 44.45 49.53))
     (stroke (width 0) (type default))
   )
-  (wire (pts (xy 63.881 32.766) (xy 64.008 32.766))
+  (wire (pts (xy 58.42 24.13) (xy 58.42 30.48))
     (stroke (width 0) (type default))
   )
-  (wire (pts (xy 39.37 50.8) (xy 48.641 50.8))
+  (wire (pts (xy 34.29 39.37) (xy 44.45 39.37))
     (stroke (width 0) (type default))
   )
-  (wire (pts (xy 39.37 48.26) (xy 48.641 48.26))
+  (wire (pts (xy 34.29 44.45) (xy 44.45 44.45))
     (stroke (width 0) (type default))
   )
-  (wire (pts (xy 48.641 40.64) (xy 48.641 40.386))
+  (wire (pts (xy 34.29 46.99) (xy 44.45 46.99))
     (stroke (width 0) (type default))
   )
-  (wire (pts (xy 39.37 53.34) (xy 48.641 53.34))
+  (wire (pts (xy 34.29 41.91) (xy 44.45 41.91))
     (stroke (width 0) (type default))
   )
-  (wire (pts (xy 48.641 45.72) (xy 48.641 45.339))
-    (stroke (width 0) (type default))
+  (text "nfault needs\npull up >2.2v at start" (at 54.61 45.72 0)
+    (effects (font (size 1.27 1.27)) (justify left bottom))
   )
-  (wire (pts (xy 39.37 55.88) (xy 48.641 55.88))
-    (stroke (width 0) (type default))
+  (text "DRVOFF turns off \nmotors when HIGH" (at 54.61 52.07 0)
+    (effects (font (size 1.27 1.27)) (justify left bottom))
   )
-  (wire (pts (xy 39.37 43.18) (xy 48.641 43.18))
-    (stroke (width 0) (type default))
-  )
-  (wire (pts (xy 63.881 28.956) (xy 63.881 32.766))
-    (stroke (width 0) (type default))
-  )
-  (wire (pts (xy 39.37 40.64) (xy 48.641 40.64))
-    (stroke (width 0) (type default))
-  )
-  (wire (pts (xy 48.641 43.18) (xy 48.641 42.926))
-    (stroke (width 0) (type default))
-  )
-  (wire (pts (xy 48.641 48.26) (xy 48.641 47.879))
-    (stroke (width 0) (type default))
+  (text "nsleep makes device \nenter sleepmode when LOW" (at 50.8 57.15 0)
+    (effects (font (size 1.27 1.27)) (justify left bottom))
   )
   (text "2" (at 269.24 194.31 0)
     (effects (font (size 1.27 1.27)) (justify left bottom))
   )
-  (symbol (lib_id "Connector_Generic:Conn_01x07") (at 34.29 48.26 0) (mirror y) (unit 1)
+  (symbol (lib_id "Connector_Generic:Conn_01x07") (at 29.21 41.91 0) (mirror y) (unit 1)
     (in_bom yes) (on_board yes) (dnp no)
-    (property "Reference" "J3" (at 34.29 61.976 0)
+    (property "Reference" "J1" (at 29.21 55.88 0)
       (effects (font (size 1.27 1.27)))
     )
-    (property "Value" "Conn_01x07" (at 34.29 59.436 0)
+    (property "Value" "Conn_01x07" (at 29.21 53.34 0)
       (effects (font (size 1.27 1.27)))
     )
-    (property "Footprint" "Connector_Molex:Molex_CLIK-Mate_502382-0770_1x07-1MP_P1.25mm_Vertical" (at 34.29 48.26 0)
+    (property "Footprint" "Connector_Molex:Molex_KK-254_AE-6410-07A_1x07_P2.54mm_Vertical" (at 29.21 41.91 0)
       (effects (font (size 1.27 1.27)) hide)
     )
-    (property "Datasheet" "~" (at 34.29 48.26 0)
+    (property "Datasheet" "~" (at 29.21 41.91 0)
       (effects (font (size 1.27 1.27)) hide)
     )
+    (pin "1")
+    (pin "7")
     (pin "5")
-    (pin "1")
+    (pin "4")
+    (pin "3")
     (pin "2")
-    (pin "4")
     (pin "6")
-    (pin "3")
-    (pin "7")
-    (instances
-      (project "driver_seperate"
-        (path "/8aa936d6-33ab-4874-8145-d1c763a0b8a3"
-          (reference "J3") (unit 1)
-        )
-      )
-    )
-  )
-  (symbol (lib_id "Connector_Generic:Conn_01x03") (at 66.421 23.876 90) (unit 1)
-    (in_bom yes) (on_board yes) (dnp no) (fields_autoplaced)
-    (property "Reference" "J1" (at 71.12 22.606 90)
-      (effects (font (size 1.27 1.27)) (justify right))
-    )
-    (property "Value" "Conn_01x03" (at 71.12 25.146 90)
-      (effects (font (size 1.27 1.27)) (justify right))
-    )
-    (property "Footprint" "Connector_Molex:Molex_CLIK-Mate_502443-0370_1x03-1MP_P2.00mm_Vertical" (at 66.421 23.876 0)
-      (effects (font (size 1.27 1.27)) hide)
-    )
-    (property "Datasheet" "~" (at 66.421 23.876 0)
-      (effects (font (size 1.27 1.27)) hide)
-    )
-    (pin "3")
-    (pin "1")
-    (pin "2")
     (instances
       (project "driver_seperate"
@@
     )
   )
-  (sheet (at 48.641 32.766) (size 36.449 28.829) (fields_autoplaced)
+  (symbol (lib_id "Connector_Generic:Conn_01x02") (at 58.42 19.05 90) (unit 1)
+    (in_bom yes) (on_board yes) (dnp no) (fields_autoplaced)
+    (property "Reference" "J4" (at 64.008 17.78 90)
+      (effects (font (size 1.27 1.27)) (justify right))
+    )
+    (property "Value" "Conn_01x02" (at 64.008 20.32 90)
+      (effects (font (size 1.27 1.27)) (justify right))
+    )
+    (property "Footprint" "Connector_Molex:Molex_KK-254_AE-6410-02A_1x02_P2.54mm_Vertical" (at 58.42 19.05 0)
+      (effects (font (size 1.27 1.27)) hide)
+    )
+    (property "Datasheet" "~" (at 58.42 19.05 0)
+      (effects (font (size 1.27 1.27)) hide)
+    )
+    (pin "2")
+    (pin "1")
+    (instances
+      (project "driver_seperate"
+        (path "/8aa936d6-33ab-4874-8145-d1c763a0b8a3"
+          (reference "J4") (unit 1)
+        )
+      )
+    )
+  )
+  (sheet (at 44.45 30.48) (size 33.02 27.94) (fields_autoplaced)
     (stroke (width 0.1524) (type solid))
     (fill (color 0 0 0 0.0000))
-    (property "Sheetname" "controller" (at 48.641 32.0544 0)
+    (property "Sheetname" "Motor Driver" (at 44.45 29.7684 0)
       (effects (font (size 1.27 1.27)) (justify left bottom))
     )
-    (property "Sheetfile" "controller.kicad_sch" (at 48.641 62.1796 0)
+    (property "Sheetfile" "controller.kicad_sch" (at 44.45 59.0046 0)
       (effects (font (size 1.27 1.27)) (justify left top))
     )
-    (pin "GND" input (at 68.961 32.766 90)
+    (pin "FGOUT" input (at 44.45 36.83 180)
+      (effects (font (size 1.27 1.27)) (justify left))
+    )
+    (pin "DIR" input (at 44.45 39.37 180)
+      (effects (font (size 1.27 1.27)) (justify left))
+    )
+    (pin "PWM" input (at 44.45 34.29 180)
+      (effects (font (size 1.27 1.27)) (justify left))
+    )
+    (pin "nSleep" input (at 44.45 49.53 180)
+      (effects (font (size 1.27 1.27)) (justify left))
+    )
+    (pin "DRVOFF" input (at 44.45 46.99 180)
+      (effects (font (size 1.27 1.27)) (justify left))
+    )
+    (pin "nFault" input (at 44.45 44.45 180)
+      (effects (font (size 1.27 1.27)) (justify left))
+    )
+    (pin "BRAKE" input (at 44.45 41.91 180)
+      (effects (font (size 1.27 1.27)) (justify left))
+    )
+    (pin "VCC" input (at 58.42 30.48 90)
       (effects (font (size 1.27 1.27)) (justify right))
     )
-    (pin "VCC" input (at 64.008 32.766 90)
+    (pin "GND" input (at 60.96 30.48 90)
       (effects (font (size 1.27 1.27)) (justify right))
     )
-    (pin "PWM" input (at 48.641 50.546 180)
-      (effects (font (size 1.27 1.27)) (justify left))
-    )
-    (pin "FGOUT" input (at 48.641 53.34 180)
-      (effects (font (size 1.27 1.27)) (justify left))
-    )
-    (pin "+3V3" passive (at 66.421 32.766 90)
-      (effects (font (size 1.27 1.27)) (justify right))
-    )
-    (pin "NRST" input (at 48.641 55.88 180)
-      (effects (font (size 1.27 1.27)) (justify left))
-    )
-    (pin "CS" input (at 48.641 47.879 180)
-      (effects (font (size 1.27 1.27)) (justify left))
-    )
-    (pin "MOSI" input (at 48.641 42.926 180)
-      (effects (font (size 1.27 1.27)) (justify left))
-    )
-    (pin "MISO" output (at 48.641 45.339 180)
-      (effects (font (size 1.27 1.27)) (justify left))
-    )
-    (pin "SCK" input (at 48.641 40.386 180)
-      (effects (font (size 1.27 1.27)) (justify left))
-    )
     (instances

Commit message: Add new design
Parts:
- removed J1: Conn_01x07, Connector_Molex:Molex_KK-254_AE-6410-07A_1x07_P2.54mm_Vertical, symbol Connector_Generic:Conn_01x07
- added H1, H2: MountingHole, MountingHole:MountingHole_3.2mm_M3, symbol Mechanical:MountingHole
- added J3: Conn_01x05, Connector_Molex:Molex_KK-254_AE-6410-05A_1x05_P2.54mm_Vertical, symbol Connector_Generic:Conn_01x05
- J4: footprint Connector_Molex:Molex_KK-254_AE-6410-02A_1x02_P2.54mm_Vertical -> Connector_Molex:Molex_KK-396_5273-02A_1x02_P3.96mm_Vertical
Connections:
- net Motor Driver/BRAKE: now also J3.2 (Pin_2)
- net Motor Driver/DIR: now also J3.3 (Pin_3)
- net Motor Driver/FGOUT: now also J3.4 (Pin_4)
- net Motor Driver/PWM: now also J3.5 (Pin_5)
- net Motor Driver/nFault: now also J3.1 (Pin_1)
Other:
- sheet Motor Driver ports: added none; removed DRVOFF, nSleep
Changed lines of the file:
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@@
     (stroke (width 0) (type default))
   )
-  (wire (pts (xy 34.29 49.53) (xy 44.45 49.53))
+  (wire (pts (xy 34.29 44.45) (xy 44.45 44.45))
     (stroke (width 0) (type default))
   )
@@
   )
   (wire (pts (xy 34.29 39.37) (xy 44.45 39.37))
-    (stroke (width 0) (type default))
-  )
-  (wire (pts (xy 34.29 44.45) (xy 44.45 44.45))
-    (stroke (width 0) (type default))
-  )
-  (wire (pts (xy 34.29 46.99) (xy 44.45 46.99))
     (stroke (width 0) (type default))
   )
@@
     (effects (font (size 1.27 1.27)) (justify left bottom))
   )
-  (symbol (lib_id "Connector_Generic:Conn_01x07") (at 29.21 41.91 0) (mirror y) (unit 1)
-    (in_bom yes) (on_board yes) (dnp no)
-    (property "Reference" "J1" (at 29.21 55.88 0)
-      (effects (font (size 1.27 1.27)))
+  (symbol (lib_id "Mechanical:MountingHole") (at 39.878 25.654 0) (unit 1)
+    (in_bom yes) (on_board yes) (dnp no) (fields_autoplaced)
+    (property "Reference" "H1" (at 43.18 24.384 0)
+      (effects (font (size 1.27 1.27)) (justify left))
     )
-    (property "Value" "Conn_01x07" (at 29.21 53.34 0)
-      (effects (font (size 1.27 1.27)))
+    (property "Value" "MountingHole" (at 43.18 26.924 0)
+      (effects (font (size 1.27 1.27)) (justify left))
     )
-    (property "Footprint" "Connector_Molex:Molex_KK-254_AE-6410-07A_1x07_P2.54mm_Vertical" (at 29.21 41.91 0)
+    (property "Footprint" "MountingHole:MountingHole_3.2mm_M3" (at 39.878 25.654 0)
       (effects (font (size 1.27 1.27)) hide)
     )
-    (property "Datasheet" "~" (at 29.21 41.91 0)
+    (property "Datasheet" "~" (at 39.878 25.654 0)
       (effects (font (size 1.27 1.27)) hide)
     )
-    (pin "1")
-    (pin "7")
-    (pin "5")
-    (pin "4")
-    (pin "3")
-    (pin "2")
-    (pin "6")
     (instances
       (project "driver_seperate"
         (path "/8aa936d6-33ab-4874-8145-d1c763a0b8a3"
-          (reference "J1") (unit 1)
+          (reference "H1") (unit 1)
+        )
+      )
+    )
+  )
+  (symbol (lib_id "Mechanical:MountingHole") (at 80.518 60.706 0) (unit 1)
+    (in_bom yes) (on_board yes) (dnp no) (fields_autoplaced)
+    (property "Reference" "H2" (at 83.82 59.436 0)
+      (effects (font (size 1.27 1.27)) (justify left))
+    )
+    (property "Value" "MountingHole" (at 83.82 61.976 0)
+      (effects (font (size 1.27 1.27)) (justify left))
+    )
+    (property "Footprint" "MountingHole:MountingHole_3.2mm_M3" (at 80.518 60.706 0)
+      (effects (font (size 1.27 1.27)) hide)
+    )
+    (property "Datasheet" "~" (at 80.518 60.706 0)
+      (effects (font (size 1.27 1.27)) hide)
+    )
+    (instances
+      (project "driver_seperate"
+        (path "/8aa936d6-33ab-4874-8145-d1c763a0b8a3"
+          (reference "H2") (unit 1)
         )
       )
@@
       (effects (font (size 1.27 1.27)) (justify right))
     )
-    (property "Footprint" "Connector_Molex:Molex_KK-254_AE-6410-02A_1x02_P2.54mm_Vertical" (at 58.42 19.05 0)
+    (property "Footprint" "Connector_Molex:Molex_KK-396_5273-02A_1x02_P3.96mm_Vertical" (at 58.42 19.05 0)
       (effects (font (size 1.27 1.27)) hide)
     )
@@
         (path "/8aa936d6-33ab-4874-8145-d1c763a0b8a3"
           (reference "J4") (unit 1)
+        )
+      )
+    )
+  )
+  (symbol (lib_id "Connector_Generic:Conn_01x05") (at 29.21 39.37 180) (unit 1)
+    (in_bom yes) (on_board yes) (dnp no) (fields_autoplaced)
+    (property "Reference" "J3" (at 29.21 27.94 0)
+      (effects (font (size 1.27 1.27)))
+    )
+    (property "Value" "Conn_01x05" (at 29.21 30.48 0)
+      (effects (font (size 1.27 1.27)))
+    )
+    (property "Footprint" "Connector_Molex:Molex_KK-254_AE-6410-05A_1x05_P2.54mm_Vertical" (at 29.21 39.37 0)
+      (effects (font (size 1.27 1.27)) hide)
+    )
+    (property "Datasheet" "~" (at 29.21 39.37 0)
+      (effects (font (size 1.27 1.27)) hide)
+    )
+    (pin "4")
+    (pin "5")
+    (pin "1")
+    (pin "2")
+    (pin "3")
+    (instances
+      (project "driver_seperate"
+        (path "/8aa936d6-33ab-4874-8145-d1c763a0b8a3"
+          (reference "J3") (unit 1)
         )
       )
@@
       (effects (font (size 1.27 1.27)) (justify left))
     )
-    (pin "nSleep" input (at 44.45 49.53 180)
-      (effects (font (size 1.27 1.27)) (justify left))
-    )
-    (pin "DRVOFF" input (at 44.45 46.99 180)
-      (effects (font (size 1.27 1.27)) (justify left))
-    )
-    (pin "nFault" input (at 44.45 44.45 180)
-      (effects (font (size 1.27 1.27)) (justify left))
-    )
     (pin "BRAKE" input (at 44.45 41.91 180)
       (effects (font (size 1.27 1.27)) (justify left))
@@
       (effects (font (size 1.27 1.27)) (justify right))
     )
+    (pin "nFault" input (at 44.45 44.45 180)
+      (effects (font (size 1.27 1.27)) (justify left))
+    )
     (instances

Commit message: Add screw holes
Parts:
- H1, H2: footprint MountingHole:MountingHole_3.2mm_M3 -> MountingHole:MountingHole_2.2mm_M2
Changed lines of the file:
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@@
       (effects (font (size 1.27 1.27)) (justify left))
     )
-    (property "Footprint" "MountingHole:MountingHole_3.2mm_M3" (at 39.878 25.654 0)
+    (property "Footprint" "MountingHole:MountingHole_2.2mm_M2" (at 39.878 25.654 0)
       (effects (font (size 1.27 1.27)) hide)
     )
@@
       (effects (font (size 1.27 1.27)) (justify left))
     )
-    (property "Footprint" "MountingHole:MountingHole_3.2mm_M3" (at 80.518 60.706 0)
+    (property "Footprint" "MountingHole:MountingHole_2.2mm_M2" (at 80.518 60.706 0)
       (effects (font (size 1.27 1.27)) hide)
     )

Commit message: Add pcb v2, Remove old files
Parts:
- J3: footprint Connector_Molex:Molex_KK-254_AE-6410-05A_1x05_P2.54mm_Vertical -> Connector_PinSocket_2.54mm:PinSocket_2x03_P2.54mm_Vertical
Changed lines of the file:
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@@
       (effects (font (size 1.27 1.27)))
     )
-    (property "Footprint" "Connector_Molex:Molex_KK-254_AE-6410-05A_1x05_P2.54mm_Vertical" (at 29.21 39.37 0)
+    (property "Footprint" "Connector_PinSocket_2.54mm:PinSocket_2x03_P2.54mm_Vertical" (at 29.21 39.37 0)
       (effects (font (size 1.27 1.27)) hide)
     )
