File: driver/driver_seperate/controller.kicad_sch (KiCad schematic)
At the start: 17 parts, among them IC1 MCT8316Z0TQRGFRQ1, J2 Motor

Commit message: Add new footprint to schematic
Parts:
- C4: footprint Capacitor_SMD:C_0805_2012Metric -> SamacSys_Parts:CAPC6153X500N
Changed lines of the file:
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@@
       (effects (font (size 1.27 1.27)) (justify left))
     )
-    (property "Footprint" "Capacitor_SMD:C_0805_2012Metric" (at 163.957 51.943 0)
+    (property "Footprint" "SamacSys_Parts:CAPC6153X500N" (at 163.957 51.943 0)
       (effects (font (size 1.27 1.27)) hide)
     )
