File: driver_seperate/driver_seperate.kicad_pcb (KiCad board)
At the start: 4 copper layers, 37.8 x 34.2 mm, 21 parts, among them IC1 MCT8316Z0TQRGFRQ1, J2 Motor, J3 Conn_01x05, J4 Conn_01x02

Commit message: Remove unused from schematic
Parts:
- C1: value 0u1F -> 100nF
- J3: value Conn_01x05 -> Connector_PinSocket_2.54mm:PinSocket_2x03_P2.54mm_Vertical
- J4: value Conn_01x02 -> Connector_Molex:Molex_KK-396_5273-02A_1x02_P3.96mm_Vertical
Connections:
- net GND renamed GNDREF
Changed lines of the file:
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@@
   (net 0 "")
   (net 1 "Net-(IC1-ILIM)")
-  (net 2 "GND")
+  (net 2 "GNDREF")
   (net 3 "/Motor Driver/VM")
   (net 4 "/Motor Driver/SW_BK")
@@
       (net 3 "/Motor Driver/VM") (pintype "passive"))
     (pad "2" smd rect (at 0.7 0 90) (size 0.78 0.98) (layers "F.Cu" "F.Paste" "F.Mask")
-      (net 2 "GND") (pintype "passive"))
+      (net 2 "GNDREF") (pintype "passive"))
     (model "C:\\Users\\anton\\projects\\seegoals\\Electronics\\driver\\SamacSys_Parts.3dshapes\\C0603C104K1RACAUTO.stp"
       (offset (xyz 0 0 0))
@@
       (net 4 "/Motor Driver/SW_BK") (pintype "passive"))
     (pad "2" smd roundrect (at 1.475 0 270) (size 1.15 1.8) (layers "F.Cu" "F.Paste" "F.Mask") (roundrect_rratio 0.2173913043)
-      (net 2 "GND") (pintype "passive"))
+      (net 2 "GNDREF") (pintype "passive"))
     (model "${KICAD6_3DMODEL_DIR}/Capacitor_SMD.3dshapes/C_1206_3216Metric.wrl"
       (offset (xyz 0 0 0))
@@
         (effects (font (size 1 1) (thickness 0.15)))
     )
-    (fp_text value "0u1F" (at 0 1.68) (layer "F.Fab")
+    (fp_text value "100nF" (at 0 1.68) (layer "F.Fab")
         (effects (font (size 1 1) (thickness 0.15)))
     )
@@
       (net 1 "Net-(IC1-ILIM)") (pintype "passive"))
     (pad "2" smd roundrect (at 0.95 0) (size 1 1.45) (layers "F.Cu" "F.Paste" "F.Mask") (roundrect_rratio 0.25)
-      (net 2 "GND") (pintype "passive"))
+      (net 2 "GNDREF") (pintype "passive"))
     (model "${KICAD6_3DMODEL_DIR}/Capacitor_SMD.3dshapes/C_0805_2012Metric.wrl"
       (offset (xyz 0 0 0))
@@
       (net 19 "/Motor Driver/W") (pinfunction "W") (pintype "passive"))
     (pad "4" thru_hole oval (at 7.62 0 180) (size 1.74 2.19) (drill 1.19) (layers "*.Cu" "*.Mask")
-      (net 2 "GND") (pinfunction "GND_BK") (pintype "passive"))
+      (net 2 "GNDREF") (pinfunction "GND_BK") (pintype "passive"))
     (pad "5" thru_hole oval (at 10.16 0 180) (size 1.74 2.19) (drill 1.19) (layers "*.Cu" "*.Mask")
       (net 21 "/Motor Driver/H2") (pinfunction "H2") (pintype "passive"))
@@
       (net 1 "Net-(IC1-ILIM)") (pintype "passive"))
     (pad "2" smd roundrect (at 0.9125 0) (size 0.975 0.95) (layers "F.Cu" "F.Paste" "F.Mask") (roundrect_rratio 0.25)
-      (net 2 "GND") (pintype "passive"))
+      (net 2 "GNDREF") (pintype "passive"))
     (model "${KICAD6_3DMODEL_DIR}/Resistor_SMD.3dshapes/R_0603_1608Metric.wrl"
       (offset (xyz 0 0 0))
@@
         (effects (font (size 1 1) (thickness 0.15)))
     )
-    (fp_text value "Conn_01x05" (at -1.27 7.85) (layer "F.Fab")
+    (fp_text value "Connector_PinSocket_2.54mm:PinSocket_2x03_P2.54mm_Vertical" (at -1.27 7.85) (layer "F.Fab")
         (effects (font (size 1 1) (thickness 0.15)))
     )
@@
         (effects (font (size 1 1) (thickness 0.15)))
     )
-    (fp_text value "Conn_01x02" (at 1.98 6.35) (layer "F.Fab")
+    (fp_text value "Connector_Molex:Molex_KK-396_5273-02A_1x02_P3.96mm_Vertical" (at 1.98 6.35) (layer "F.Fab")
         (effects (font (size 1 1) (thickness 0.15)))
     )
@@
       (net 3 "/Motor Driver/VM") (pinfunction "Pin_1") (pintype "passive"))
     (pad "2" thru_hole oval (at 3.96 0) (size 3.16 4.2) (drill 1.8) (layers "*.Cu" "*.Mask")
-      (net 2 "GND") (pinfunction "Pin_2") (pintype "passive"))
+      (net 2 "GNDREF") (pinfunction "Pin_2") (pintype "passive"))
     (model "${KICAD6_3DMODEL_DIR}/Connector_Molex.3dshapes/Molex_KK-396_5273-02A_1x02_P3.96mm_Vertical.wrl"
       (offset (xyz 0 0 0))
@@
       (net 6 "/Motor Driver/AVDD") (pintype "passive"))
     (pad "2" smd rect (at 1.4 0) (size 1.02 1.82) (layers "F.Cu" "F.Paste" "F.Mask")
-      (net 2 "GND") (pintype "passive"))
+      (net 2 "GNDREF") (pintype "passive"))
     (model "C:\\Users\\anton\\projects\\seegoals\\Electronics\\driver\\SamacSys_Parts.3dshapes\\KAF31GR72A105KL.stp"
       (offset (xyz 0 0 0))
@@
     (property "Sheetname" "Motor Driver")
     (property "Voltage" ">=48v")
-    (property "ki_description" "Polarized capacitor, small symbol")
+    (property "ki_description" "Unpolarized capacitor")
     (property "ki_keywords" "cap capacitor")
     (attr smd)
@@
       (net 3 "/Motor Driver/VM") (pintype "passive"))
     (pad "2" smd rect (at 2.53 0) (size 1.86 5.52) (layers "F.Cu" "F.Paste" "F.Mask")
-      (net 2 "GND") (pintype "passive"))
+      (net 2 "GNDREF") (pintype "passive"))
     (model "KCM55TR71H226MH01L.stp"
       (offset (xyz 0 0 0))
@@
       (net 11 "unconnected-(IC1-NC-Pad1)") (pinfunction "NC") (pintype "no_connect"))
     (pad "2" smd rect (at -2.5 -2.25 270) (size 0.3 0.8) (layers "F.Cu" "F.Paste" "F.Mask")
-      (net 2 "GND") (pinfunction "AGND_1") (pintype "passive"))
+      (net 2 "GNDREF") (pinfunction "AGND_1") (pintype "passive"))
     (pad "3" smd rect (at -2.5 -1.75 270) (size 0.3 0.8) (layers "F.Cu" "F.Paste" "F.Mask")
       (net 4 "/Motor Driver/SW_BK") (pinfunction "FB_BK") (pintype "passive"))
     (pad "4" smd rect (at -2.5 -1.25 270) (size 0.3 0.8) (layers "F.Cu" "F.Paste" "F.Mask")
-      (net 2 "GND") (pinfunction "GND_BK") (pintype "passive"))
+      (net 2 "GNDREF") (pinfunction "GND_BK") (pintype "passive"))
     (pad "5" smd rect (at -2.5 -0.75 270) (size 0.3 0.8) (layers "F.Cu" "F.Paste" "F.Mask")
       (net 12 "Net-(IC1-SW_BK)") (pinfunction "SW_BK") (pintype "passive"))
@@
       (net 3 "/Motor Driver/VM") (pinfunction "VM_3") (pintype "passive"))
     (pad "12" smd rect (at -2.5 2.75 270) (size 0.3 0.8) (layers "F.Cu" "F.Paste" "F.Mask")
-      (net 2 "GND") (pinfunction "PGND_1") (pintype "passive"))
+      (net 2 "GNDREF") (pinfunction "PGND_1") (pintype "passive"))
     (pad "13" smd rect (at -1.75 3.5 180) (size 0.3 0.8) (layers "F.Cu" "F.Paste" "F.Mask")
       (net 9 "/Motor Driver/U") (pinfunction "OUTA_1") (pintype "passive"))
@@
       (net 9 "/Motor Driver/U") (pinfunction "OUTA_2") (pintype "passive"))
     (pad "15" smd rect (at -0.75 3.5 180) (size 0.3 0.8) (layers "F.Cu" "F.Paste" "F.Mask")
-      (net 2 "GND") (pinfunction "PGND_2") (pintype "passive"))
+      (net 2 "GNDREF") (pinfunction "PGND_2") (pintype "passive"))
     (pad "16" smd rect (at -0.25 3.5 180) (size 0.3 0.8) (layers "F.Cu" "F.Paste" "F.Mask")
       (net 10 "/Motor Driver/V") (pinfunction "OUTB_1") (pintype "passive"))
@@
       (net 10 "/Motor Driver/V") (pinfunction "OUTB_2") (pintype "passive"))
     (pad "18" smd rect (at 0.75 3.5 180) (size 0.3 0.8) (layers "F.Cu" "F.Paste" "F.Mask")
-      (net 2 "GND") (pinfunction "PGND_3") (pintype "passive"))
+      (net 2 "GNDREF") (pinfunction "PGND_3") (pintype "passive"))
     (pad "19" smd rect (at 1.25 3.5 180) (size 0.3 0.8) (layers "F.Cu" "F.Paste" "F.Mask")
       (net 19 "/Motor Driver/W") (pinfunction "OUTC_1") (pintype "passive"))
@@
       (net 19 "/Motor Driver/W") (pinfunction "OUTC_2") (pintype "passive"))
     (pad "21" smd rect (at 2.5 2.75 270) (size 0.3 0.8) (layers "F.Cu" "F.Paste" "F.Mask")
-      (net 2 "GND") (pinfunction "DRVOFF") (pintype "passive"))
+      (net 2 "GNDREF") (pinfunction "DRVOFF") (pintype "passive"))
     (pad "22" smd rect (at 2.5 2.25 270) (size 0.3 0.8) (layers "F.Cu" "F.Paste" "F.Mask")
       (net 27 "/Motor Driver/nFault") (pinfunction "NFAULT") (pintype "passive"))
@@
       (net 6 "/Motor Driver/AVDD") (pinfunction "AVDD") (pintype "passive"))
     (pad "26" smd rect (at 2.5 0.25 270) (size 0.3 0.8) (layers "F.Cu" "F.Paste" "F.Mask")
-      (net 2 "GND") (pinfunction "AGND_2") (pintype "passive"))
+      (net 2 "GNDREF") (pinfunction "AGND_2") (pintype "passive"))
     (pad "27" smd rect (at 2.5 -0.25 270) (size 0.3 0.8) (layers "F.Cu" "F.Paste" "F.Mask")
       (net 20 "/Motor Driver/H1") (pinfunction "HPA") (pintype "passive"))
@@
       (net 26 "/Motor Driver/FGOUT") (pinfunction "FGOUT") (pintype "passive"))
     (pad "41" smd rect (at 0 0 180) (size 3.8 5.8) (layers "F.Cu" "F.Paste" "F.Mask")
-      (net 2 "GND") (pinfunction "EP") (pintype "passive"))
+      (net 2 "GNDREF") (pinfunction "EP") (pintype "passive"))
     (model "C:\\Users\\anton\\projects\\seegoals\\Electronics\\driver\\SamacSys_Parts.3dshapes\\MCT8316Z0TQRGFRQ1.stp"
       (offset (xyz 0 0 0))
@@
     )
   )
-  (zone (net 2) (net_name "GND") (layer "F.Cu") (hatch edge 0.5)
+  (zone (net 2) (net_name "GNDREF") (layer "F.Cu") (hatch edge 0.5)
     (priority 1)
     (connect_pads yes (clearance 0.3))
@@
     )
   )
-  (zone (net 2) (net_name "GND") (layer "F.Cu") (hatch edge 0.5)
+  (zone (net 2) (net_name "GNDREF") (layer "F.Cu") (hatch edge 0.5)
     (priority 3)
     (connect_pads (clearance 0.5))
@@
     )
   )
-  (zone (net 2) (net_name "GND") (layer "In1.Cu") (hatch edge 0.5)
+  (zone (net 2) (net_name "GNDREF") (layer "In1.Cu") (hatch edge 0.5)
     (priority 5)
     (connect_pads (clearance 0.5))
