File: kicker_v1/kicker_v1.kicad_pcb (KiCad board)
At the start: 2 copper layers, 140 x 85.3 mm, 71 parts, among them IC1 SI8620EC-B-IS, IC10 MCP1790, IC3 ADC122S051, IC4 MCP9701A, IC6 MCP6002, IC7 LT3751FE, IC8 FAN3229TMX, Q1 FDS2582, Q2 IKB40N65ES5, Q3 IKB40N65ES5, X1 DF13-12P-1.25V

Commit message: File structure enhanced.
Added uniform titleblocks and 3D renders for easier view, file cleanups.
Other:
- board text added: "Routings was modified majorly, more via's added and few placement modifications For viewing 3d, enable virtual model in 3d view"
