File: pwr_v2/pwr_v2.kicad_pcb (KiCad board)
At the start: 4 copper layers, 166 x 166 mm, 78 parts, among them CN11 Conn_02x36_Odd_Even, CN12 Conn_02x36_Odd_Even, J1 Conn_01x12_Pin, M1 Conn_02x03_Counter_Clockwise, M2 Conn_02x03_Counter_Clockwise, M3 Conn_02x03_Counter_Clockwise, M4 Conn_02x03_Counter_Clockwise, Q1 BUK9832-55A, Q2 BSS84, SW1 SW_SPST, U1 LM2576S-5, U2 LM2576S-12, U3 LM2576S-3.3, U4 LSM6DSLTR

Commit message: File structure enhanced.
Added uniform titleblocks and 3D renders for easier view, file cleanups.
Other:
- board text removed: "0"
- board text removed: "0 mm"
- board text removed: "0.01 mm"
- board text removed: "0.02"
- board text removed: "0.035 mm"
- board text removed: "0.1 mm"
- board text removed: "0.3000 mm"
- board text removed: "0.3048 mm / 0.1500 mm"
- board text removed: "1"
- board text removed: "1.24 mm"
- board text removed: "1.6000 mm"
- board text removed: "165.9975 mm x 166.0050 mm"
- board text removed: "3.3"
- board text removed: "4"
- board text removed: "4.5"
- board text removed: "B.Cu"
- board text removed: "B.Mask"
- board text removed: "B.Paste"
- board text removed: "B.Silkscreen"
- board text removed: "BOARD CHARACTERISTICS"
- board text removed: "Board Thickness:"
- board text removed: "Board overall dimensions:"
- board text removed: "Bottom Silk Screen"
- board text removed: "Bottom Solder Mask"
- board text removed: "Bottom Solder Paste"
- board text removed: "Castellated pads:"
- board text removed: "Color"
- board text removed: "Copper Finish:"
- board text removed: "Copper Layer Count:"
- board text removed: "Dielectric"
- board text removed: "Edge card connectors:"
- board text removed: "Epsilon R"
- board text removed: "F.Cu"
- board text removed: "F.Mask"
- board text removed: "F.Paste"
- board text removed: "F.Silkscreen"
- board text removed: "FR4"
- board text removed: "Impedance Control:"
- board text removed: "In1.Cu"
- board text removed: "In2.Cu"
- board text removed: "Layer Name"
- board text removed: "Loss Tangent"
- board text removed: "Material"
- board text removed: "Min hole diameter:"
- board text removed: "Min track/spacing:"
- board text removed: "No"
- board text removed: "None"
- board text removed: "Not specified"
- board text removed: "Plated Board Edge:"
- board text removed: "Thickness (mm)"
- board text removed: "Top Silk Screen"
- board text removed: "Top Solder Mask"
- board text removed: "Top Solder Paste"
- board text removed: "Type"
- board text removed: "copper"
- board text removed: "core"
- board text removed: "prepreg"
